Commit message: Update.

File: src/airobot/urdfs/yumi_grippers.original.urdf (robot description, URDF)
Before this commit: robot yumi, 22 links, 21 joints
Links:
- added link table_top; visual mesh filename=meshes/table/table_top.stl
Joints:
- added joint yumi_body_to_table_top: type fixed, parent yumi_body, child table_top, origin xyz=0.110910 0 0.0 rpy=0 0 1.57079
